File: project/pimo.kicad_sch (KiCad schematic)
At the start: 10 parts, among them J1 RPi_GPIO, J11 Conn_01x03_Pin, J2 Conn_01x05_Pin, J3 Conn_ARM_JTAG_SWD_10, U1 W25Q32JVSS

Commit message: added most of the things.
Parts:
- added J4: Conn_01x01, Connector_PinHeader_1.27mm:PinHeader_1x01_P1.27mm_Vertical, symbol Connector_Generic:Conn_01x01
- J2: footprint (none) -> Connector_PinHeader_2.54mm:PinHeader_1x05_P2.54mm_Vertical
- J3: footprint (none) -> Connector_PinHeader_1.27mm:PinHeader_2x05_P1.27mm_Vertical
Connections:
- net RESET is gone; now on net ~{RESET}: A1.15 (GPIO11)
- net GND: now also J3.3 (GND), J3.5 (GND)
- net RTCK: now also J4.1 (Pin_1)
- net VTref: now reaches J3.1 (VTref)
- net ~{RESET}: now reaches J3.10 (~{RESET})
- net SWDIO/TMS: now reaches J3.2 (SWDIO/TMS)
- net SWCLK/TCK: now reaches J3.4 (SWCLK/TCK)
- net SWO/TDO: now reaches J3.6 (SWO/TDO)
- net NC/TDI: now reaches J3.8 (NC/TDI)
- net GNDDetect: now reaches J3.9 (GNDDetect)
Other:
- moved on the sheet: C1, C2, J11, J3, U1

Commit message: smaller spi footprint
Parts:
- U1: footprint Package_SO:SOIC-8_5.23x5.23mm_P1.27mm -> Package_SO:SOIC-8_3.9x4.9mm_P1.27mm
Changed lines of the file:
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@@
 			)
 		)
-		(property "Footprint" "Package_SO:SOIC-8_5.23x5.23mm_P1.27mm"
+		(property "Footprint" "Package_SO:SOIC-8_3.9x4.9mm_P1.27mm"
 			(at 63.5 166.37 0)
 			(effects

Commit message: bonus jtag header
Parts:
- added J5: Conn_01x05_Pin, Connector_PinHeader_2.54mm:PinHeader_1x05_P2.54mm_Vertical, symbol Connector:Conn_01x05_Pin
Connections:
- net GND: now also J5.5 (Pin_5)
- net GNDDetect: now also J5.2 (Pin_2)
- net RTCK: now also J5.1 (Pin_1)
- net VTref: now also J5.4 (Pin_4)
- net pico3v3 renamed 3V3
- net 3V3: now also J5.3 (Pin_3)
Other:
- moved on the sheet: J3, J4

Commit message: pmod header.  v1.1
Parts:
- added J6: 2.54-2*6P Bend insert, TinyTapeout_PMOD:PinHeader_2x06_P2.54mm_PMODPeriph2B, symbol tt:PMOD_PERIPH_2x6
- added R2: 1k, Resistor_SMD:R_0603_1608Metric, symbol Device:R_Small
Connections:
- net GND: now also J6.11 (GND), J6.5 (GND); no longer A1.29 (GPIO22), D1.2 (A), R1.1, R1.2
- net PMOD1_IN: now reaches J11.2 (Pin_2), U1.1 (~{CS})
- net PMOD1_IN: now also J6.1 (IO1), R2.2
- net PMOD5: now reaches U1.3 (IO2)
- net PMOD5: now also J6.7 (IO5)
- net PMOD6: now reaches U1.7 (IO3)
- net PMOD6: now also J6.8 (IO6)
- net 3V3 renamed +3.3V
- net +3.3V: now also J6.12 (VCC), J6.6 (VCC), R2.1
- net RPI_SPI_CLK renamed PMOD4
- net PMOD4: now also J6.4 (IO4)
- net RPI_SPI_MISO renamed PMOD3
- net PMOD3: now also J6.3 (IO3)
- net RPI_SPI_MOSI renamed PMOD2
- net PMOD2: now also J6.2 (IO2)
- new net: D1.2 (A), R1.1
- new net: A1.29 (GPIO22), R1.2
- new net PMOD7_IN: J6.9 (IO7)
- new net PMOD8_IN: J6.10 (IO8)
Other:
- note added: "PMOD"
- moved on the sheet: C1, C2, D1, J3, J4, J5, R1, U1
